File: proximity/proximity.sch (KiCad schematic (older format))
At the start: 34 parts, among them IC1 NRF51822, P1 CONN_3X2, P2 ST-0503, P3 AIN_0_3, P4 AIN_4_7, Q1 MOSFET_N, SW1 SWITCH-4, SW2 SWITCH-4, U1 ANTENNA-NC, X1 FOX924

Commit message: nRF51822 proximity tag updates: - Ordinary crystal instead of CMOS oscillator - Regular pin header for SWDIO and SWCLK
Parts:
- removed D4: DIODE, symbol DIODE
- removed P1: CONN_3X2, symbol CONN_3X2
- removed P2: ST-0503, symbol CONN_2
- removed Q1: MOSFET_N, symbol MOSFET_N
- removed R4: 100R, symbol R
- removed R5: 10K, symbol R
- added C5, C6: 12pF, ~, symbol C
- added P1: CONN_2, ~, symbol CONN_2
- X1: value FOX924 -> NX2520SA
Connections:
- net labels removed: BUZZER
- wire segments 145 -> 135
- no-connect marks 17 -> 14
