File: cam85/cam85.kicad_pcb (KiCad board)
At the start: 2 copper layers, 18.4 x 22.2 mm, 14 parts, among them IC1 ATTINY85-S, P1 CONN_2, P2 CONN_2, P3 CONN_3X2, P4 CONN_2, P5 CONN_2, Q1 MOSFET_N, Q2 MOSFET_N, SW1 SWITCH_INV

Commit message: Redesign for optocouplers
Parts:
- removed Q1, Q2: MOSFET_N, SOT23GDS
- added IC2: MOCD207M, SOIC8-3.9MM, F.Cu at (29.2, 27.3)
- added R2: 200R, SM0603, F.Cu at (34.8, 29.0)
- added R3: 200R, SM0603, F.Cu at (34.8, 25.9)
- P4, P5: footprint WIREWRAP-PIN-2 -> PIN_ARRAY_2X1
- moved P5 8.47 mm to (26.7, 34.3)
- moved P4 6.63 mm to (30.5, 38.1), turned to 0 degrees
- renumbered P1 to BAT
Connections:
- net /DOUT renamed /CAMPOW
Routing:
- net N-0000014: track 5.09 -> 13.7 mm, vias 0 -> 1
- net N-000008: track 4.99 -> 13.5 mm
- net N-0000017: track 4.20 -> 10.8 mm, vias 0 -> 1
- net N-000001: track 5.86 -> 11.2 mm
- net VCC: track 25.9 -> 30.4 mm
- net N-0000016: track 0.00 -> 3.35 mm
- net N-0000018: track 0.00 -> 2.93 mm
- net GND: track 7.66 -> 9.91 mm, vias 1 -> 2
- net /STRBTN: track 9.79 -> 8.92 mm, vias 2 -> 0
- net /PWRBTN: track 5.45 -> 6.28 mm, vias 2 -> 0
- net /RESET: track 15.6 -> 15.0 mm
Other:
- board size 18.4 x 22.2 mm -> 21 x 22.2 mm
- board text added: "Spy camera shutter timer"
