File: cam85/cam85.sch (KiCad schematic (older format))
At the start: 14 parts, among them IC1 ATTINY85-S, P1 CONN_2, P2 CONN_2, P3 CONN_3X2, P4 CONN_2, P5 CONN_2, Q1 MOSFET_N, Q2 MOSFET_N, SW1 SWITCH_INV

Commit message: Redesign for optocouplers
Parts:
- removed Q1, Q2: MOSFET_N, symbol MOSFET_N
- added IC2: MOCD207M, symbol MOCD207M
- added R2, R3: 200R, symbol R
Connections:
- net labels added: CAMPOW
- net labels removed: DOUT
- wire segments 40 -> 42
Other:
- moved on the sheet: P4
Changed lines of the file:
@@
-EESchema Schematic File Version 2  date Fri 25 Jan 2013 11:46:50 AM EST
+EESchema Schematic File Version 2  date Fri 08 Feb 2013 08:35:11 PM EST
+LIBS:guan
 LIBS:power
 LIBS:device
@@
 Sheet 1 1
 Title ""
-Date "25 jan 2013"
+Date "9 feb 2013"
 Rev ""
 Comp ""
@@
 Wire Wire Line
 	1800 2200 2300 2200
-$Comp
-L MOSFET_N Q1
-U 1 1 5101F466
-P 3700 3800
-F 0 "Q1" H 3710 3970 60  0000 R CNN
-F 1 "MOSFET_N" H 3710 3650 60  0000 R CNN
-	1    3700 3800
-	1    0    0    -1
-$EndComp
-$Comp
-L MOSFET_N Q2
-U 1 1 5102A5A0
-P 5700 3800
-F 0 "Q2" H 5710 3970 60  0000 R CNN
-F 1 "MOSFET_N" H 5710 3650 60  0000 R CNN
-	1    5700 3800
-	1    0    0    -1
-$EndComp
 Text Label 1800 2100 0    60   ~ 0
 PWRBTN
@@
 OUTLED
 Text Label 1300 1900 0    60   ~ 0
-DOUT
+CAMPOW
 $Comp
 L C C1
@@
 Wire Wire Line
 	2100 3600 2600 3600
-Text Label 2350 3600 0    60   ~ 0
-DOUT
+Text Label 2250 3600 0    60   ~ 0
+CAMPOW
 $Comp
 L GND #PWR05
@@
 	3200 2900 3300 2900
 NoConn ~ 3200 3100
-Wire Wire Line
-	5100 3800 5500 3800
-Wire Wire Line
-	3100 3800 3500 3800
-Text Label 3100 3800 0    60   ~ 0
+Text Label 3550 4400 0    60   ~ 0
 PWRBTN
-Text Label 5100 3800 0    60   ~ 0
-STRBTN
 $Comp
 L CONN_2 P4
 U 1 1 5102B1F2
-P 4350 3800
-F 0 "P4" V 4300 3800 40  0000 C CNN
-F 1 "CONN_2" V 4400 3800 40  0000 C CNN
-	1    4350 3800
-	1    0    0    -1
-$EndComp
+P 5300 5250
+F 0 "P4" V 5250 5250 40  0000 C CNN
+F 1 "CONN_2" V 5350 5250 40  0000 C CNN
+	1    5300 5250
+	1    0    0    -1
+$EndComp
+$Comp
+L MOCD207M IC2
+U 1 1 5115A798
+P 4450 5250
+F 0 "IC2" H 4450 4900 60  0000 C CNN
+F 1 "MOCD207M" H 4400 5600 60  0000 C CNN
+	1    4450 5250
+	1    0    0    -1
+$EndComp
+Wire Wire Line
+	4950 5150 4950 5000
+Wire Wire Line
+	4950 5350 4950 5500
+$Comp
+L R R2
+U 1 1 5115A829
+P 3950 4650
+F 0 "R2" V 4030 4650 50  0000 C CNN
+F 1 "200R" V 3950 4650 50  0000 C CNN
+	1    3950 4650
+	1    0    0    -1
+$EndComp
+Wire Wire Line
+	3950 4900 3950 5000
+$Comp
+L GND #PWR07
+U 1 1 5115A85D
+P 3850 5600
+F 0 "#PWR07" H 3850 5600 30  0001 C CNN
+F 1 "GND" H 3850 5530 30  0001 C CNN
+	1    3850 5600
+	1    0    0    -1
+$EndComp
+Wire Wire Line
+	3850 5600 3850 5500
+Wire Wire Line
+	3850 5500 3950 5500
+Wire Wire Line
+	3950 4400 3550 4400
+Text Label 5500 4400 0    60   ~ 0
+STRBTN
 $Comp
 L CONN_2 P5
-U 1 1 5102B201
-P 6350 3800
-F 0 "P5" V 6300 3800 40  0000 C CNN
-F 1 "CONN_2" V 6400 3800 40  0000 C CNN
-	1    6350 3800
-	1    0    0    -1
-$EndComp
-Wire Wire Line
-	5800 3600 6000 3600
-Wire Wire Line
-	6000 3600 6000 3700
-Wire Wire Line
-	5800 4000 6000 4000
-Wire Wire Line
-	6000 4000 6000 3900
-Wire Wire Line
-	3800 3600 4000 3600
-Wire Wire Line
-	4000 3600 4000 3700
-Wire Wire Line
-	3800 4000 4000 4000
-Wire Wire Line
-	4000 4000 4000 3900
+U 1 1 5115AB88
+P 7250 5250
+F 0 "P5" V 7200 5250 40  0000 C CNN
+F 1 "CONN_2" V 7300 5250 40  0000 C CNN
+	1    7250 5250
+	1    0    0    -1
+$EndComp
+$Comp
+L MOCD207M IC2
+U 2 1 5115AB8E
+P 6400 5250
+F 0 "IC2" H 6400 4900 60  0000 C CNN
+F 1 "MOCD207M" H 6350 5600 60  0000 C CNN
+	2    6400 5250
+	1    0    0    -1
+$EndComp
+Wire Wire Line
+	6900 5150 6900 5000
+Wire Wire Line
+	6900 5350 6900 5500
+$Comp
+L R R3
+U 1 1 5115AB96
+P 5900 4650
+F 0 "R3" V 5980 4650 50  0000 C CNN
+F 1 "200R" V 5900 4650 50  0000 C CNN
+	1    5900 4650
+	1    0    0    -1
+$EndComp
+Wire Wire Line
+	5900 4900 5900 5000
+$Comp
+L GND #PWR08
+U 1 1 5115AB9D
+P 5800 5600
+F 0 "#PWR08" H 5800 5600 30  0001 C CNN
+F 1 "GND" H 5800 5530 30  0001 C CNN
+	1    5800 5600
+	1    0    0    -1
+$EndComp
+Wire Wire Line
+	5800 5600 5800 5500
+Wire Wire Line
+	5800 5500 5900 5500
+Wire Wire Line
+	5900 4400 5500 4400
 $EndSCHEMATC
