File: shoe/shoe.sch (KiCad schematic (older format))
At the start: 28 parts, among them IC1 ATMEGA328P-A, IC2 TLC5940-PWP, K1 CONN_3, P1 CONN_2, P10 CONN_2, P11 CONN_2, P12 CONN_2, P13 CONN_2, P14 CONN_2, P15 CONN_2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

Commit message: Shoe board v2
- Add PTC fuse and reverse protection shunt diode
- Replace IR section (because of timer conflict) with exposed serial
Parts:
- removed C3: 0.1uF, symbol C
- removed R1: 10K, symbol R
- added D?: DIODE, symbol DIODE
- added F?: FUSE, symbol FUSE
Connections:
- net labels added: RX, TX
- net labels removed: IR
- wire segments 97 -> 101
- no-connect marks 19 -> 18
Other:
- moved on the sheet: K1
Changed lines of the file:
@@
-EESchema Schematic File Version 2  date Thu 21 Feb 2013 09:08:56 AM EST
+EESchema Schematic File Version 2  date Thu 21 Feb 2013 09:18:02 AM EST
 LIBS:guan
 LIBS:power
@@
 Sheet 1 1
 Title ""
-Date "4 dec 2012"
+Date "21 feb 2013"
 Rev ""
 Comp ""
@@
 Wire Wire Line
 	900  5600 1400 5600
-Connection ~ 2700 5800
-Wire Wire Line
-	2700 5900 2700 5800
-Wire Wire Line
-	2400 5700 3000 5700
-Wire Wire Line
-	4000 2950 4500 2950
-Wire Wire Line
-	4800 3550 4900 3550
 Wire Wire Line
 	4000 2300 4500 2300
@@
 Wire Wire Line
 	4300 3550 4000 3550
-Wire Wire Line
-	3000 5600 2500 5600
-Wire Wire Line
-	2400 5800 3000 5800
-Wire Wire Line
-	2700 6400 2700 6300
 Wire Wire Line
 	900  5800 1400 5800
@@
 	1    1200 6100
 	1    0    0    -1
-$EndComp
-$Comp
-L VCC #PWR019
-U 1 1 50BCF7BA
-P 900 5800
-F 0 "#PWR019" H 900 5900 30  0001 C CNN
-F 1 "VCC" H 900 5900 30  0000 C CNN
-F 2 "" H 900 5800 60  0001 C CNN
-F 3 "" H 900 5800 60  0001 C CNN
-	1    900  5800
-	0    -1   -1   0
 $EndComp
 $Comp
@@
 $EndComp
 $Comp
-L GND #PWR021
-U 1 1 50BCF7A7
-P 2700 6400
-F 0 "#PWR021" H 2700 6400 30  0001 C CNN
-F 1 "GND" H 2700 6330 30  0001 C CNN
-F 2 "" H 2700 6400 60  0001 C CNN
-F 3 "" H 2700 6400 60  0001 C CNN
-	1    2700 6400
-	1    0    0    -1
-$EndComp
-$Comp
-L C C3
-U 1 1 50BCF7A3
-P 2700 6100
-F 0 "C3" H 2750 6200 50  0000 L CNN
-F 1 "0.1uF" H 2750 6000 50  0000 L CNN
-F 2 "" H 2700 6100 60  0001 C CNN
-F 3 "" H 2700 6100 60  0001 C CNN
-	1    2700 6100
-	1    0    0    -1
-$EndComp
-$Comp
-L VCC #PWR022
-U 1 1 50BCF796
-P 2400 5800
-F 0 "#PWR022" H 2400 5900 30  0001 C CNN
-F 1 "VCC" H 2400 5900 30  0000 C CNN
-F 2 "" H 2400 5800 60  0001 C CNN
-F 3 "" H 2400 5800 60  0001 C CNN
-	1    2400 5800
-	0    -1   -1   0
-$EndComp
-$Comp
-L GND #PWR023
-U 1 1 50BCF791
-P 2400 5700
-F 0 "#PWR023" H 2400 5700 30  0001 C CNN
-F 1 "GND" H 2400 5630 30  0001 C CNN
-F 2 "" H 2400 5700 60  0001 C CNN
-F 3 "" H 2400 5700 60  0001 C CNN
-	1    2400 5700
-	0    1    1    0
-$EndComp
-Text Label 2500 5600 0    60   ~ 0
-IR
-$Comp
 L CONN_3 K1
 U 1 1 50BCF781
-P 3350 5700
-F 0 "K1" V 3300 5700 50  0000 C CNN
-F 1 "CONN_3" V 3400 5700 40  0000 C CNN
-F 2 "" H 3350 5700 60  0001 C CNN
-F 3 "" H 3350 5700 60  0001 C CNN
-	1    3350 5700
-	1    0    0    -1
+P 2650 5700
+F 0 "K1" V 2600 5700 50  0000 C CNN
+F 1 "CONN_3" V 2700 5700 40  0000 C CNN
+F 2 "" H 2650 5700 60  0001 C CNN
+F 3 "" H 2650 5700 60  0001 C CNN
+	1    2650 5700
+	-1   0    0    1
 $EndComp
 NoConn ~ 4000 3350
@@
 NoConn ~ 4000 3150
 NoConn ~ 4000 3050
-Text Label 4400 2950 0    60   ~ 0
-IR
 NoConn ~ 4000 4400
 NoConn ~ 4000 4300
@@
 NoConn ~ 4000 4100
 NoConn ~ 4000 3900
-NoConn ~ 4000 3800
-NoConn ~ 4000 3700
 Text Label 4100 3550 0    60   ~ 0
 RESET
-$Comp
-L R R1
-U 1 1 50BCF757
-P 4550 3550
-F 0 "R1" V 4630 3550 50  0000 C CNN
-F 1 "10K" V 4550 3550 50  0000 C CNN
-F 2 "" H 4550 3550 60  0001 C CNN
-F 3 "" H 4550 3550 60  0001 C CNN
-	1    4550 3550
-	0    -1   -1   0
-$EndComp
-$Comp
-L VCC #PWR024
-U 1 1 50BCF752
-P 4900 3550
-F 0 "#PWR024" H 4900 3650 30  0001 C CNN
-F 1 "VCC" H 4900 3650 30  0000 C CNN
-F 2 "" H 4900 3550 60  0001 C CNN
-F 3 "" H 4900 3550 60  0001 C CNN
-	1    4900 3550
-	0    1    1    0
-$EndComp
 Text Label 4250 4000 0    60   ~ 0
 GSCLK
@@
 GSCLK
 $Comp
-L GND #PWR025
+L GND #PWR021
 U 1 1 50BCF698
 P 8400 2500
-F 0 "#PWR025" H 8400 2500 30  0001 C CNN
+F 0 "#PWR021" H 8400 2500 30  0001 C CNN
 F 1 "GND" H 8400 2430 30  0001 C CNN
 F 2 "" H 8400 2500 60  0001 C CNN
@@
 $EndComp
 $Comp
-L VCC #PWR026
+L VCC #PWR022
 U 1 1 50BCF63B
 P 6100 1700
-F 0 "#PWR026" H 6100 1800 30  0001 C CNN
+F 0 "#PWR022" H 6100 1800 30  0001 C CNN
 F 1 "VCC" H 6100 1800 30  0000 C CNN
 F 2 "" H 6100 1700 60  0001 C CNN
@@
 BLANK
 $Comp
-L GND #PWR027
+L GND #PWR023
 U 1 1 50BCF61E
 P 6000 2900
-F 0 "#PWR027" H 6000 2900 30  0001 C CNN
+F 0 "#PWR023" H 6000 2900 30  0001 C CNN
 F 1 "GND" H 6000 2830 30  0001 C CNN
 F 2 "" H 6000 2900 60  0001 C CNN
@@
 SCLK
 $Comp
-L GND #PWR028
+L GND #PWR024
 U 1 1 50BCF5BF
 P 5950 2400
-F 0 "#PWR028" H 5950 2400 30  0001 C CNN
+F 0 "#PWR024" H 5950 2400 30  0001 C CNN
 F 1 "GND" H 5950 2330 30  0001 C CNN
 F 2 "" H 5950 2400 60  0001 C CNN
@@
 $EndComp
 $Comp
-L GND #PWR029
+L GND #PWR025
 U 1 1 50BCF5B6
 P 8100 2300
-F 0 "#PWR029" H 8100 2300 30  0001 C CNN
+F 0 "#PWR025" H 8100 2300 30  0001 C CNN
 F 1 "GND" H 8100 2230 30  0001 C CNN
 F 2 "" H 8100 2300 60  0001 C CNN
@@
 $EndComp
 $Comp
-L VCC #PWR030
+L VCC #PWR026
 U 1 1 50BCF5AE
 P 7500 2200
-F 0 "#PWR030" H 7500 2300 30  0001 C CNN
+F 0 "#PWR026" H 7500 2300 30  0001 C CNN
 F 1 "VCC" H 7500 2300 30  0000 C CNN
 F 2 "" H 7500 2200 60  0001 C CNN
@@
 LED15
 $Comp
-L GND #PWR031
+L GND #PWR027
 U 1 1 50BCF531
 P 1900 4500
-F 0 "#PWR031" H 1900 4500 30  0001 C CNN
+F 0 "#PWR027" H 1900 4500 30  0001 C CNN
 F 1 "GND" H 1900 4430 30  0001 C CNN
 F 2 "" H 1900 4500 60  0001 C CNN
@@
 NoConn ~ 2100 3450
 $Comp
-L GND #PWR032
+L GND #PWR028
 U 1 1 50BCF4F3
 P 1300 2400
-F 0 "#PWR032" H 1300 2400 30  0001 C CNN
+F 0 "#PWR028" H 1300 2400 30  0001 C CNN
 F 1 "GND" H 1300 2330 30  0001 C CNN
 F 2 "" H 1300 2400 60  0001 C CNN
@@
 $EndComp
 $Comp
-L VCC #PWR033
+L VCC #PWR029
 U 1 1 50BCF4E6
 P 1900 2000
-F 0 "#PWR033" H 1900 2100 30  0001 C CNN
+F 0 "#PWR029" H 1900 2100 30  0001 C CNN
 F 1 "VCC" H 1900 2100 30  0000 C CNN
 F 2 "" H 1900 2000 60  0001 C CNN
@@
 	1    0    0    -1
 $EndComp
+$Comp
+L GND #PWR030
+U 1 1 51262CD5
+P 3100 5900
+F 0 "#PWR030" H 3100 5900 30  0001 C CNN
+F 1 "GND" H 3100 5830 30  0001 C CNN
+F 2 "" H 3100 5900 60  0000 C CNN
+F 3 "" H 3100 5900 60  0000 C CNN
+	1    3100 5900
+	1    0    0    -1
+$EndComp
+Wire Wire Line
+	3000 5800 3100 5800
+Wire Wire Line
+	3100 5800 3100 5900
+Wire Wire Line
+	3000 5700 3250 5700
+Wire Wire Line
+	3000 5600 3250 5600
+Text Label 3100 5700 0    60   ~ 0
+RX
+Text Label 3100 5600 0    60   ~ 0
+TX
+NoConn ~ 4000 2950
+Wire Wire Line
+	4000 3700 4500 3700
+Wire Wire Line
+	4000 3800 4500 3800
+Text Label 4350 3700 0    60   ~ 0
+RX
+Text Label 4350 3800 0    60   ~ 0
+TX
+$Comp
+L FUSE F?
+U 1 1 51263141
+P 900 6050
+F 0 "F?" H 1000 6100 40  0000 C CNN
+F 1 "FUSE" H 800 6000 40  0000 C CNN
+F 2 "" H 900 6050 60  0000 C CNN
+F 3 "" H 900 6050 60  0000 C CNN
+	1    900  6050
+	0    -1   -1   0
+$EndComp
+$Comp
+L VCC #PWR?
+U 1 1 51263150
+P 750 6300
+F 0 "#PWR?" H 750 6400 30  0001 C CNN
+F 1 "VCC" H 750 6400 30  0000 C CNN
+F 2 "" H 750 6300 60  0000 C CNN
+F 3 "" H 750 6300 60  0000 C CNN
+	1    750  6300
+	0    -1   -1   0
+$EndComp
+Wire Wire Line
+	750  6300 900  6300
+$Comp
+L DIODE D?
+U 1 1 512631C9
+P 700 5700
+F 0 "D?" H 700 5800 40  0000 C CNN
+F 1 "DIODE" H 700 5600 40  0000 C CNN
+F 2 "" H 700 5700 60  0000 C CNN
+F 3 "" H 700 5700 60  0000 C CNN
+	1    700  5700
+	0    1    1    0
+$EndComp
+Wire Wire Line
+	700  5500 1100 5500
+Wire Wire Line
+	1100 5500 1100 5600
+Connection ~ 1100 5600
+Wire Wire Line
+	700  5900 800  5900
+Wire Wire Line
+	800  5900 800  6300
+Connection ~ 800  6300
 $EndSCHEMATC

Commit message: shoe updates
Parts:
- gave numbers to parts that had none: 2
Changed lines of the file:
@@
-EESchema Schematic File Version 2  date Thu 21 Feb 2013 09:18:02 AM EST
+EESchema Schematic File Version 2  date Thu 21 Feb 2013 09:32:01 AM EST
 LIBS:guan
 LIBS:power
@@
 $EndComp
 $Comp
-L GND #PWR020
+L GND #PWR019
 U 1 1 50BCF7B7
 P 900 5600
-F 0 "#PWR020" H 900 5600 30  0001 C CNN
+F 0 "#PWR019" H 900 5600 30  0001 C CNN
 F 1 "GND" H 900 5530 30  0001 C CNN
 F 2 "" H 900 5600 60  0001 C CNN
@@
 GSCLK
 $Comp
-L GND #PWR021
+L GND #PWR020
 U 1 1 50BCF698
 P 8400 2500
-F 0 "#PWR021" H 8400 2500 30  0001 C CNN
+F 0 "#PWR020" H 8400 2500 30  0001 C CNN
 F 1 "GND" H 8400 2430 30  0001 C CNN
 F 2 "" H 8400 2500 60  0001 C CNN
@@
 $EndComp
 $Comp
-L VCC #PWR022
+L VCC #PWR021
 U 1 1 50BCF63B
 P 6100 1700
-F 0 "#PWR022" H 6100 1800 30  0001 C CNN
+F 0 "#PWR021" H 6100 1800 30  0001 C CNN
 F 1 "VCC" H 6100 1800 30  0000 C CNN
 F 2 "" H 6100 1700 60  0001 C CNN
@@
 BLANK
 $Comp
-L GND #PWR023
+L GND #PWR022
 U 1 1 50BCF61E
 P 6000 2900
-F 0 "#PWR023" H 6000 2900 30  0001 C CNN
+F 0 "#PWR022" H 6000 2900 30  0001 C CNN
 F 1 "GND" H 6000 2830 30  0001 C CNN
 F 2 "" H 6000 2900 60  0001 C CNN
@@
 SCLK
 $Comp
-L GND #PWR024
+L GND #PWR023
 U 1 1 50BCF5BF
 P 5950 2400
-F 0 "#PWR024" H 5950 2400 30  0001 C CNN
+F 0 "#PWR023" H 5950 2400 30  0001 C CNN
 F 1 "GND" H 5950 2330 30  0001 C CNN
 F 2 "" H 5950 2400 60  0001 C CNN
@@
 $EndComp
 $Comp
-L GND #PWR025
+L GND #PWR024
 U 1 1 50BCF5B6
 P 8100 2300
-F 0 "#PWR025" H 8100 2300 30  0001 C CNN
+F 0 "#PWR024" H 8100 2300 30  0001 C CNN
 F 1 "GND" H 8100 2230 30  0001 C CNN
 F 2 "" H 8100 2300 60  0001 C CNN
@@
 $EndComp
 $Comp
-L VCC #PWR026
+L VCC #PWR025
 U 1 1 50BCF5AE
 P 7500 2200
-F 0 "#PWR026" H 7500 2300 30  0001 C CNN
+F 0 "#PWR025" H 7500 2300 30  0001 C CNN
 F 1 "VCC" H 7500 2300 30  0000 C CNN
 F 2 "" H 7500 2200 60  0001 C CNN
@@
 LED15
 $Comp
-L GND #PWR027
+L GND #PWR026
 U 1 1 50BCF531
 P 1900 4500
-F 0 "#PWR027" H 1900 4500 30  0001 C CNN
+F 0 "#PWR026" H 1900 4500 30  0001 C CNN
 F 1 "GND" H 1900 4430 30  0001 C CNN
 F 2 "" H 1900 4500 60  0001 C CNN
@@
 NoConn ~ 2100 3450
 $Comp
-L GND #PWR028
+L GND #PWR027
 U 1 1 50BCF4F3
 P 1300 2400
-F 0 "#PWR028" H 1300 2400 30  0001 C CNN
+F 0 "#PWR027" H 1300 2400 30  0001 C CNN
 F 1 "GND" H 1300 2330 30  0001 C CNN
 F 2 "" H 1300 2400 60  0001 C CNN
@@
 $EndComp
 $Comp
-L VCC #PWR029
+L VCC #PWR028
 U 1 1 50BCF4E6
 P 1900 2000
-F 0 "#PWR029" H 1900 2100 30  0001 C CNN
+F 0 "#PWR028" H 1900 2100 30  0001 C CNN
 F 1 "VCC" H 1900 2100 30  0000 C CNN
 F 2 "" H 1900 2000 60  0001 C CNN
@@
 $EndComp
 $Comp
-L GND #PWR030
+L GND #PWR029
 U 1 1 51262CD5
 P 3100 5900
-F 0 "#PWR030" H 3100 5900 30  0001 C CNN
+F 0 "#PWR029" H 3100 5900 30  0001 C CNN
 F 1 "GND" H 3100 5830 30  0001 C CNN
 F 2 "" H 3100 5900 60  0000 C CNN
@@
 TX
 $Comp
-L FUSE F?
+L FUSE F1
 U 1 1 51263141
 P 900 6050
-F 0 "F?" H 1000 6100 40  0000 C CNN
+F 0 "F1" H 1000 6100 40  0000 C CNN
 F 1 "FUSE" H 800 6000 40  0000 C CNN
 F 2 "" H 900 6050 60  0000 C CNN
@@
 $EndComp
 $Comp
-L VCC #PWR?
+L VCC #PWR030
 U 1 1 51263150
 P 750 6300
-F 0 "#PWR?" H 750 6400 30  0001 C CNN
+F 0 "#PWR030" H 750 6400 30  0001 C CNN
 F 1 "VCC" H 750 6400 30  0000 C CNN
 F 2 "" H 750 6300 60  0000 C CNN
@@
 	750  6300 900  6300
 $Comp
-L DIODE D?
+L DIODE D1
 U 1 1 512631C9
 P 700 5700
-F 0 "D?" H 700 5800 40  0000 C CNN
+F 0 "D1" H 700 5800 40  0000 C CNN
 F 1 "DIODE" H 700 5600 40  0000 C CNN
 F 2 "" H 700 5700 60  0000 C CNN
