File: charger/charger.sch (KiCad schematic (older format))
At the start: 8 parts, among them CON1 USB-MINI-B, P1 MAX1555, P2 CONN_2, P3 CONN_2, P4 CONN_2

Commit message: MAX1555 update
Parts:
- removed P4: CONN_2, symbol CONN_2
- added D1: LED, symbol LED
- added K1: CONN_3, symbol CONN_3
- added R1: 1K, symbol R
Connections:
- net labels added: 3.3V
- wire segments 28 -> 32
Changed lines of the file:
@@
-EESchema Schematic File Version 2  date Thu 21 Feb 2013 12:05:43 PM EST
+EESchema Schematic File Version 2  date Thu 21 Feb 2013 01:16:31 PM EST
 LIBS:power
 LIBS:device
@@
 LIBS:contrib
 LIBS:valves
+LIBS:charger-cache
 EELAYER 27 0
 EELAYER END
@@
 NoConn ~ 5100 2550
 $Comp
-L GND #PWR01
+L GND #PWR4
 U 1 1 51264ED5
 P 6300 2800
-F 0 "#PWR01" H 6300 2800 30  0001 C CNN
+F 0 "#PWR4" H 6300 2800 30  0001 C CNN
 F 1 "GND" H 6300 2730 30  0001 C CNN
 F 2 "" H 6300 2800 60  0000 C CNN
@@
 Connection ~ 6300 2250
 $Comp
-L GND #PWR02
+L GND #PWR1
 U 1 1 51264EF4
 P 5000 2800
-F 0 "#PWR02" H 5000 2800 30  0001 C CNN
+F 0 "#PWR1" H 5000 2800 30  0001 C CNN
 F 1 "GND" H 5000 2730 30  0001 C CNN
 F 2 "" H 5000 2800 60  0000 C CNN
@@
 $EndComp
 $Comp
-L GND #PWR03
+L GND #PWR7
 U 1 1 51264F60
 P 7300 1600
-F 0 "#PWR03" H 7300 1600 30  0001 C CNN
+F 0 "#PWR7" H 7300 1600 30  0001 C CNN
 F 1 "GND" H 7300 1530 30  0001 C CNN
 F 2 "" H 7300 1600 60  0000 C CNN
@@
 $EndComp
 $Comp
-L GND #PWR04
+L GND #PWR5
 U 1 1 51264FC7
 P 6600 1550
-F 0 "#PWR04" H 6600 1550 30  0001 C CNN
+F 0 "#PWR5" H 6600 1550 30  0001 C CNN
 F 1 "GND" H 6600 1480 30  0001 C CNN
 F 2 "" H 6600 1550 60  0000 C CNN
@@
 VUSB
 $Comp
-L GND #PWR05
+L GND #PWR6
 U 1 1 5126508B
 P 7100 2350
-F 0 "#PWR05" H 7100 2350 30  0001 C CNN
+F 0 "#PWR6" H 7100 2350 30  0001 C CNN
 F 1 "GND" H 7100 2280 30  0001 C CNN
 F 2 "" H 7100 2350 60  0000 C CNN
@@
 BAT
 $Comp
-L GND #PWR06
+L GND #PWR8
 U 1 1 5126518E
 P 8200 1600
-F 0 "#PWR06" H 8200 1600 30  0001 C CNN
+F 0 "#PWR8" H 8200 1600 30  0001 C CNN
 F 1 "GND" H 8200 1530 30  0001 C CNN
 F 2 "" H 8200 1600 60  0000 C CNN
@@
 Wire Wire Line
 	8200 1500 8300 1500
-$Comp
-L CONN_2 P4
-U 1 1 512651B4
-P 9600 1400
-F 0 "P4" V 9550 1400 40  0000 C CNN
-F 1 "CONN_2" V 9650 1400 40  0000 C CNN
-F 2 "" H 9600 1400 60  0000 C CNN
-F 3 "" H 9600 1400 60  0000 C CNN
-	1    9600 1400
-	1    0    0    -1
-$EndComp
-$Comp
-L GND #PWR07
-U 1 1 512651C3
-P 9150 1600
-F 0 "#PWR07" H 9150 1600 30  0001 C CNN
-F 1 "GND" H 9150 1530 30  0001 C CNN
-F 2 "" H 9150 1600 60  0000 C CNN
-F 3 "" H 9150 1600 60  0000 C CNN
-	1    9150 1600
-	1    0    0    -1
-$EndComp
-Wire Wire Line
-	9150 1600 9150 1500
-Wire Wire Line
-	9150 1500 9250 1500
-Wire Wire Line
-	9050 1300 9250 1300
+Wire Wire Line
+	9050 1300 9350 1300
 Text Label 9050 1300 0    60   ~ 0
 \POK
@@
 $EndComp
 $Comp
-L GND #PWR08
+L GND #PWR3
 U 1 1 51265261
 P 6250 1550
-F 0 "#PWR08" H 6250 1550 30  0001 C CNN
+F 0 "#PWR3" H 6250 1550 30  0001 C CNN
 F 1 "GND" H 6250 1480 30  0001 C CNN
 F 2 "" H 6250 1550 60  0000 C CNN
@@
 $EndComp
 $Comp
-L GND #PWR09
+L GND #PWR2
 U 1 1 512652B9
 P 5900 1550
-F 0 "#PWR09" H 5900 1550 30  0001 C CNN
+F 0 "#PWR2" H 5900 1550 30  0001 C CNN
 F 1 "GND" H 5900 1480 30  0001 C CNN
 F 2 "" H 5900 1550 60  0000 C CNN
@@
 Text Label 5900 950  0    60   ~ 0
 BAT
+$Comp
+L LED D1
+U 1 1 51266477
+P 9550 1300
+F 0 "D1" H 9550 1400 50  0000 C CNN
+F 1 "LED" H 9550 1200 50  0000 C CNN
+F 2 "" H 9550 1300 60  0000 C CNN
+F 3 "" H 9550 1300 60  0000 C CNN
+	1    9550 1300
+	-1   0    0    1
+$EndComp
+$Comp
+L R R1
+U 1 1 512664A4
+P 10100 1300
+F 0 "R1" V 10180 1300 50  0000 C CNN
+F 1 "1K" V 10100 1300 50  0000 C CNN
+F 2 "" H 10100 1300 60  0000 C CNN
+F 3 "" H 10100 1300 60  0000 C CNN
+	1    10100 1300
+	0    -1   -1   0
+$EndComp
+Wire Wire Line
+	10350 1300 10650 1300
+Text Label 10500 1300 0    60   ~ 0
+BAT
+Wire Wire Line
+	9750 1300 9850 1300
+$Comp
+L CONN_3 K1
+U 1 1 51266567
+P 9250 2400
+F 0 "K1" V 9200 2400 50  0000 C CNN
+F 1 "CONN_3" V 9300 2400 40  0000 C CNN
+F 2 "" H 9250 2400 60  0000 C CNN
+F 3 "" H 9250 2400 60  0000 C CNN
+	1    9250 2400
+	1    0    0    -1
+$EndComp
+Wire Wire Line
+	8600 2300 8900 2300
+Text Label 8600 2300 0    60   ~ 0
+BAT
+Wire Wire Line
+	8600 2400 8900 2400
+Text Label 8600 2400 0    60   ~ 0
+3.3V
+$Comp
+L GND #PWR9
+U 1 1 512665B7
+P 8800 2600
+F 0 "#PWR9" H 8800 2600 30  0001 C CNN
+F 1 "GND" H 8800 2530 30  0001 C CNN
+F 2 "" H 8800 2600 60  0000 C CNN
+F 3 "" H 8800 2600 60  0000 C CNN
+	1    8800 2600
+	1    0    0    -1
+$EndComp
+Wire Wire Line
+	8800 2600 8800 2500
+Wire Wire Line
+	8800 2500 8900 2500
 $EndSCHEMATC
