File: ltc3783/ltc3783.sch (KiCad schematic (older format))
At the start: 19 parts

Commit message: LTC3783
Connections:
- net ILIM: now also IC?.14 (OV/FB), R?.1
Changed lines of the file:
@@
-EESchema Schematic File Version 2  date Fri 22 Feb 2013 10:24:22 AM EST
+EESchema Schematic File Version 2  date Mon 04 Mar 2013 04:22:28 PM EST
 LIBS:guan
 LIBS:power
@@
 LIBS:contrib
 LIBS:valves
+LIBS:ltc3783-cache
 EELAYER 27 0
 EELAYER END
@@
 Sheet 1 1
 Title ""
-Date "22 feb 2013"
+Date "4 mar 2013"
 Rev ""
 Comp ""
@@
 Wire Wire Line
 	6500 1200 6400 1200
+Wire Wire Line
+	4450 2200 4450 2000
+Connection ~ 4450 2000
 $EndSCHEMATC
