File: vertex/vertex.sch (KiCad schematic (older format))
At the start: 5 parts, among them K1 CONN_3, K2 CONN_3, P1 CONN_6, P2 CONN_6, P3 CONN_6

Commit message: Game of Life vertex board rev1
Parts:
- removed K2: CONN_3, symbol CONN_3
- added P4, P5, P6: CONN_1, ~, symbol CONN_1
Changed lines of the file:
@@
-EESchema Schematic File Version 2  date Tue 05 Mar 2013 01:24:30 PM EST
+EESchema Schematic File Version 2  date Fri 03 May 2013 02:36:41 AM EDT
 LIBS:power
 LIBS:device
@@
 LIBS:valves
 LIBS:vertex-cache
-EELAYER 27 0
+EELAYER 24 0
 EELAYER END
 $Descr A4 11693 8268
@@
 Sheet 1 1
 Title ""
-Date "5 mar 2013"
+Date "3 may 2013"
 Rev ""
 Comp ""
@@
 $EndComp
 $Comp
-L CONN_3 K2
-U 1 1 51363401
-P 5000 4200
-F 0 "K2" V 4950 4200 50  0000 C CNN
-F 1 "CONN_3" V 5050 4200 40  0000 C CNN
-F 2 "" H 5000 4200 60  0000 C CNN
-F 3 "" H 5000 4200 60  0000 C CNN
-	1    5000 4200
-	-1   0    0    1
-$EndComp
-$Comp
 L GND #PWR010
 U 1 1 51363410
@@
 	5350 3800 5350 3700
 $Comp
-L GND #PWR011
-U 1 1 51363436
-P 5350 4400
-F 0 "#PWR011" H 5350 4400 30  0001 C CNN
-F 1 "GND" H 5350 4330 30  0001 C CNN
-F 2 "" H 5350 4400 60  0000 C CNN
-F 3 "" H 5350 4400 60  0000 C CNN
-	1    5350 4400
-	1    0    0    -1
-$EndComp
-Wire Wire Line
-	5350 4400 5350 4300
-$Comp
-L +3.3V #PWR012
-U 1 1 5136345D
-P 5450 4200
-F 0 "#PWR012" H 5450 4160 30  0001 C CNN
-F 1 "+3.3V" H 5450 4310 30  0000 C CNN
-F 2 "" H 5450 4200 60  0000 C CNN
-F 3 "" H 5450 4200 60  0000 C CNN
-	1    5450 4200
-	0    1    1    0
-$EndComp
-Wire Wire Line
-	5450 4200 5350 4200
-$Comp
-L +12V #PWR013
-U 1 1 51363485
-P 5450 4100
-F 0 "#PWR013" H 5450 4050 20  0001 C CNN
-F 1 "+12V" H 5450 4200 30  0000 C CNN
-F 2 "" H 5450 4100 60  0000 C CNN
-F 3 "" H 5450 4100 60  0000 C CNN
-	1    5450 4100
-	0    1    1    0
-$EndComp
-Wire Wire Line
-	5450 4100 5350 4100
-$Comp
-L +3.3V #PWR014
+L +3.3V #PWR011
 U 1 1 513634AE
 P 5450 3600
-F 0 "#PWR014" H 5450 3560 30  0001 C CNN
+F 0 "#PWR011" H 5450 3560 30  0001 C CNN
 F 1 "+3.3V" H 5450 3710 30  0000 C CNN
 F 2 "" H 5450 3600 60  0000 C CNN
@@
 	5450 3600 5350 3600
 $Comp
-L +12V #PWR015
+L +12V #PWR012
 U 1 1 513634D8
 P 5450 3500
-F 0 "#PWR015" H 5450 3450 20  0001 C CNN
+F 0 "#PWR012" H 5450 3450 20  0001 C CNN
 F 1 "+12V" H 5450 3600 30  0000 C CNN
 F 2 "" H 5450 3500 60  0000 C CNN
@@
 Wire Wire Line
 	5450 3500 5350 3500
+$Comp
+L CONN_1 P4
+U 1 1 518137BA
+P 6650 3600
+F 0 "P4" H 6730 3600 40  0000 L CNN
+F 1 "CONN_1" H 6650 3655 30  0001 C CNN
+F 2 "~" H 6650 3600 60  0000 C CNN
+F 3 "~" H 6650 3600 60  0000 C CNN
+	1    6650 3600
+	1    0    0    -1
+$EndComp
+$Comp
+L CONN_1 P5
+U 1 1 518137C9
+P 6650 3700
+F 0 "P5" H 6730 3700 40  0000 L CNN
+F 1 "CONN_1" H 6650 3755 30  0001 C CNN
+F 2 "~" H 6650 3700 60  0000 C CNN
+F 3 "~" H 6650 3700 60  0000 C CNN
+	1    6650 3700
+	1    0    0    -1
+$EndComp
+$Comp
+L CONN_1 P6
+U 1 1 51813846
+P 6650 3800
+F 0 "P6" H 6730 3800 40  0000 L CNN
+F 1 "CONN_1" H 6650 3855 30  0001 C CNN
+F 2 "~" H 6650 3800 60  0000 C CNN
+F 3 "~" H 6650 3800 60  0000 C CNN
+	1    6650 3800
+	1    0    0    -1
+$EndComp
 $EndSCHEMATC
