File: vertex/vertex.sch (KiCad schematic (older format))
At the start: 7 parts, among them K1 CONN_3, P1 CONN_6, P2 CONN_6, P3 CONN_6, P4 CONN_1, P5 CONN_1, P6 CONN_1

Commit message: Hack Manhattan Color Life boards final version
Connections:
- net +12V: now also P1.4, P2.4, P3.4; no longer P1.3, P2.3, P3.3
- net +3.3V: now also P1.5, P2.5, P3.5; no longer P1.2, P2.2, P3.2
- net GND: now also P1.6, P2.6, P3.6; no longer P1.1, P2.1, P3.1
- new net: P1.3, P2.1, P3.2
- new net: P1.1, P2.2, P3.3
- new net: P1.2, P2.3, P3.1
Other:
- moved on the sheet: P1, P2, P3
Changed lines of the file:
@@
-EESchema Schematic File Version 2  date Fri 10 May 2013 01:00:30 PM EDT
+EESchema Schematic File Version 2
 LIBS:power
 LIBS:device
@@
 Sheet 1 1
 Title ""
-Date "3 may 2013"
+Date "23 may 2013"
 Rev ""
 Comp ""
@@
 L CONN_6 P2
 U 1 1 512EA817
-P 5050 1750
-F 0 "P2" V 5000 1750 60  0000 C CNN
-F 1 "CONN_6" V 5100 1750 60  0000 C CNN
-F 2 "" H 5050 1750 60  0000 C CNN
-F 3 "" H 5050 1750 60  0000 C CNN
-	1    5050 1750
-	0    -1   -1   0
+P 5050 2450
+F 0 "P2" V 5000 2450 60  0000 C CNN
+F 1 "CONN_6" V 5100 2450 60  0000 C CNN
+F 2 "" H 5050 2450 60  0000 C CNN
+F 3 "" H 5050 2450 60  0000 C CNN
+	1    5050 2450
+	0    1    1    0
 $EndComp
 $Comp
 L CONN_6 P1
 U 1 1 512EA826
-P 4150 2750
-F 0 "P1" V 4100 2750 60  0000 C CNN
-F 1 "CONN_6" V 4200 2750 60  0000 C CNN
-F 2 "" H 4150 2750 60  0000 C CNN
-F 3 "" H 4150 2750 60  0000 C CNN
-	1    4150 2750
-	-1   0    0    1
+P 4850 2750
+F 0 "P1" V 4800 2750 60  0000 C CNN
+F 1 "CONN_6" V 4900 2750 60  0000 C CNN
+F 2 "" H 4850 2750 60  0000 C CNN
+F 3 "" H 4850 2750 60  0000 C CNN
+	1    4850 2750
+	1    0    0    -1
 $EndComp
 $Comp
 L CONN_6 P3
 U 1 1 512EA835
-P 5950 2750
-F 0 "P3" V 5900 2750 60  0000 C CNN
-F 1 "CONN_6" V 6000 2750 60  0000 C CNN
-F 2 "" H 5950 2750 60  0000 C CNN
-F 3 "" H 5950 2750 60  0000 C CNN
-	1    5950 2750
-	1    0    0    -1
+P 5250 2750
+F 0 "P3" V 5200 2750 60  0000 C CNN
+F 1 "CONN_6" V 5300 2750 60  0000 C CNN
+F 2 "" H 5250 2750 60  0000 C CNN
+F 3 "" H 5250 2750 60  0000 C CNN
+	1    5250 2750
+	-1   0    0    1
 $EndComp
 $Comp
